Commit message: gazebo works with rgbd now + todo: fix color image in rviz

File: ros2_ws/src/diff_drive_robot/urdf/robot.gazebo.xacro (robot description, xacro)
@@ -24,39 +24,46 @@
         </plugin>
     </gazebo>
-    <!-- LiDAR (PointCloud2) -->
-    <gazebo reference="laser_frame">
-        <sensor type="gpu_ray" name="lidar_sensor">
+    <!-- RGBD Camera (depth + color) -->
+    <gazebo reference="camera_frame">
+        <sensor type="depth" name="depth_sensor">
             <pose>0 0 0 0 0 0</pose>
             <visualize>true</visualize>
             <update_rate>10.0</update_rate>
-            <ray>
-                <scan>
-                    <horizontal>
-                        <samples>1800</samples>
-                        <resolution>1.0</resolution>
-                        <min_angle>-3.14159</min_angle>
-                        <max_angle>3.14159</max_angle>
-                    </horizontal>
-                    <vertical>
-                        <samples>16</samples>
-                        <resolution>2.0</resolution>
-                        <min_angle>-0.2793</min_angle>
-                        <max_angle>0.2443</max_angle>
-                    </vertical>
-                </scan>
-                <range>
-                    <min>0.2</min>
-                    <max>30.0</max>
-                    <resolution>0.01</resolution>
-                </range>
-                <noise>
-                    <type>gaussian</type>
-                    <mean>0.0</mean>
-                    <stddev>0.008</stddev>
-                </noise>
-                <output_type>point_cloud</output_type>
-            </ray>
-            <topic>pointcloud</topic>
-            <frame_name>laser_frame</frame_name>
+            <camera>
+                <image>
+                    <width>640</width>
+                    <height>480</height>
+                    <format>R_FLOAT32</format>
+                </image>
+                <clip>
+                    <near>0.2</near>
+                    <far>30.0</far>
+                </clip>
+                <horizontal_fov>1.047</horizontal_fov> <!-- 60 градусов -->
+                <vertical_fov>0.785</vertical_fov>    <!-- 45 градусов -->
+            </camera>
+            <topic>camera/depth/image_raw</topic>
+            <frame_name>camera_depth_frame</frame_name>
+            <output_type>image</output_type>
+        </sensor>
+        <sensor type="camera" name="color_sensor">
+            <pose>0 0 0 0 0 0</pose>
+            <visualize>true</visualize>
+            <update_rate>10.0</update_rate>
+            <camera>
+                <image>
+                    <width>640</width>
+                    <height>480</height>
+                    <format>RGB_INT8</format>
+                </image>
+                <clip>
+                    <near>0.2</near>
+                    <far>30.0</far>
+                </clip>
+                <horizontal_fov>1.047</horizontal_fov>
+                <vertical_fov>0.785</vertical_fov>
+            </camera>
+            <topic>camera/color/image_raw</topic>
+            <frame_name>camera_color_frame</frame_name>
         </sensor>
     </gazebo>

File: ros2_ws/src/diff_drive_robot/urdf/robot.xacro (robot description, xacro)
@@ -123,11 +123,11 @@
         <mu2>1.0</mu2>
     </gazebo>
-    <!-- Lidar link (visual only) -->
-    <joint name="laser_joint" type="fixed">
+    <!-- RGBD Camera link visuals -->
+    <joint name="camera_joint" type="fixed">
         <parent link="chassis"/>
-        <child link="laser_frame"/>
+        <child link="camera_frame"/>
         <origin xyz="0.1 0 0.175" rpy="0 0 0"/>
     </joint>
-    <link name="laser_frame">
+    <link name="camera_frame">
         <visual>
             <origin xyz="0 0 0"/>
@@ -135,5 +135,5 @@
                 <cylinder length="0.04" radius="0.05"/>
             </geometry>
-            <material name="laser_material">
+            <material name="camera_material">
                 <color rgba="0.13 0.13 0.13 1.0"/>
             </material>

Commit message: fixed rgbd + fixed gz plugins

File: ros2_ws/src/diff_drive_robot/urdf/robot.gazebo.xacro (robot description, xacro)
@@ -25,45 +25,24 @@
     </gazebo>
     <!-- RGBD Camera (depth + color) -->
-    <gazebo reference="camera_frame">
-        <sensor type="depth" name="depth_sensor">
-            <pose>0 0 0 0 0 0</pose>
-            <visualize>true</visualize>
-            <update_rate>10.0</update_rate>
-            <camera>
-                <image>
-                    <width>640</width>
-                    <height>480</height>
-                    <format>R_FLOAT32</format>
-                </image>
-                <clip>
-                    <near>0.2</near>
-                    <far>30.0</far>
-                </clip>
-                <horizontal_fov>1.047</horizontal_fov> <!-- 60 градусов -->
-                <vertical_fov>0.785</vertical_fov>    <!-- 45 градусов -->
-            </camera>
-            <topic>camera/depth/image_raw</topic>
-            <frame_name>camera_depth_frame</frame_name>
-            <output_type>image</output_type>
-        </sensor>
-        <sensor type="camera" name="color_sensor">
-            <pose>0 0 0 0 0 0</pose>
-            <visualize>true</visualize>
-            <update_rate>10.0</update_rate>
-            <camera>
-                <image>
-                    <width>640</width>
-                    <height>480</height>
-                    <format>RGB_INT8</format>
-                </image>
-                <clip>
-                    <near>0.2</near>
-                    <far>30.0</far>
-                </clip>
-                <horizontal_fov>1.047</horizontal_fov>
-                <vertical_fov>0.785</vertical_fov>
-            </camera>
-            <topic>camera/color/image_raw</topic>
-            <frame_name>camera_color_frame</frame_name>
+    <gazebo reference="camera_link">
+        <sensor name="rgbd_camera" type="rgbd_camera">
+          <gz_frame_id>camera_link</gz_frame_id>
+          <ignition_frame_id>camera_link</ignition_frame_id>
+          <camera>
+            <horizontal_fov>1.047</horizontal_fov>
+            <image>
+              <width>320</width>
+              <height>240</height>
+            </image>
+            <clip>
+              <near>0.2</near>
+              <far>100</far>
+            </clip>
+          </camera>
+          <always_on>1</always_on>
+          <update_rate>30</update_rate>
+          <visualize>true</visualize>
+          <topic>rgbd_camera</topic>
+          <enable_metrics>true</enable_metrics>
         </sensor>
     </gazebo>

File: ros2_ws/src/diff_drive_robot/urdf/robot.xacro (robot description, xacro)
@@ -126,8 +126,8 @@
     <joint name="camera_joint" type="fixed">
         <parent link="chassis"/>
-        <child link="camera_frame"/>
+        <child link="camera_link"/>
         <origin xyz="0.1 0 0.175" rpy="0 0 0"/>
     </joint>
-    <link name="camera_frame">
+    <link name="camera_link">
         <visual>
             <origin xyz="0 0 0"/>
